File: Nixie-Tube-Clock-PCB.kicad_sch (KiCad schematic)
At the start: 0 parts

Commit message: edit
Parts:
- added A1: RaspberryPi_Pico_W, Module:Raspberry_Pi_Zero_Socketed_THT_FaceDown_MountingHoles, symbol MCU_Module:RaspberryPi_Pico_W
- added ABS06-32.768KHZ-T1: Crystal Oscilator, symbol Device:Crystal
- added BT1: Battery_Cell, symbol Device:Battery_Cell
- added C1, C14, C17: 10nF, symbol Device:C
- added C10, C5, C8: 1u, symbol Device:C
- added C11: 2u, symbol Device:C
- added C12: 4.7p, symbol Device:C
- added C13, C15, C16, C18, C2, C3: 10n, symbol Device:C
- added C19, C4, C9: 0.1u, symbol Device:C
- added C6: 0.001u, symbol Device:C
- added C7: 10u, symbol Device:C
- added D1, D2, D3: D_Schottky, symbol Device:D_Schottky
- added J1, J2, J3, J4, J5, J6: Conn_01x11_Socket, symbol Connector:Conn_01x11_Socket
- added J7: Barrel_Jack_MountingPin, symbol Connector:Barrel_Jack_MountingPin
- added L1: 220u, symbol Device:L
- added R1, R2, R3: R, symbol Device:R
- added R10, R11, R12, R13, R14, R15: 5k, symbol Device:R
- added R4: 240, symbol Device:R
- added R5: 720, symbol Device:R
- added R6: 68.2k, symbol Device:R
- added R7: 100, symbol Device:R
- added R8: 1.74M, symbol Device:R
- added R9: 15k, symbol Device:R
- added U1, U10, U3: 74HC595, symbol 74xx:74HC595
- added U11, U12, U2, U7, U8, U9: ~, symbol K155ID1:K155ID1
- added U4: LM317_SOT-223, Package_TO_SOT_SMD:SOT-223-3_TabPin2, symbol Regulator_Linear:LM317_SOT-223
- added U5: DS1307N+, Package_DIP:DIP-8_W7.62mm, symbol Timer_RTC:DS1307N+
- added U6: ~, symbol LT8331:LT8331IMSE#WPBF
Connections:
- new net: J3.3 (Pin_3), U11.1 (8)
- new net: J3.4 (Pin_4), U11.10 (7)
- new net: J3.5 (Pin_5), U11.11 (6)
- new net: J3.7 (Pin_7), U11.13 (4)
- new net: J3.6 (Pin_6), U11.14 (5)
- new net: J3.10 (Pin_10), U11.15 (1)
- new net: J3.1 (Pin_1), U11.16 (0)
- new net: J3.2 (Pin_2), U11.2 (9)
- new net: U10.15 (QA), U11.3 (A)
- new net: U10.3 (QD), U11.4 (D)
- new net: U10.1 (QB), U11.6 (B)
- new net: U10.2 (QC), U11.7 (C)
- new net: J3.9 (Pin_9), U11.8 (2)
- new net: J3.8 (Pin_8), U11.9 (3)
- new net: U3.1 (QB), U8.6 (B)
- new net: U3.15 (QA), U8.3 (A)
- new net: U3.2 (QC), U8.7 (C)
- new net: U3.3 (QD), U8.4 (D)
- new net: U2.3 (A), U3.4 (QE)
- new net: U2.6 (B), U3.5 (QF)
- new net: U2.7 (C), U3.6 (QG)
- new net: U2.4 (D), U3.7 (QH)
- new net: C10.2, C11.1, D1.1 (K), R7.2
- new net: C9.2, D1.2 (A), L1.2, U6.16 (SW)
- new net: J3.11 (Pin_11), R12.2
- new net: J5.3 (Pin_3), U8.1 (8)
- new net: J5.4 (Pin_4), U8.10 (7)
- new net: J5.5 (Pin_5), U8.11 (6)
- new net: J5.7 (Pin_7), U8.13 (4)
- new net: J5.6 (Pin_6), U8.14 (5)
- new net: J5.10 (Pin_10), U8.15 (1)
- new net: J5.1 (Pin_1), U8.16 (0)
- new net: J5.2 (Pin_2), U8.2 (9)
- new net: J5.9 (Pin_9), U8.8 (2)
- new net: J5.8 (Pin_8), U8.9 (3)
- new net: R4.2, R5.1, U4.1 (ADJ)
- new net: ABS06-32.768KHZ-T1.1, U5.1 (X1)
- new net: ABS06-32.768KHZ-T1.2, U5.2 (X2)
- new net: BT1.1 (+), U5.3 (VBAT)
- new net: J2.3 (Pin_3), U7.1 (8)
- new net: J2.4 (Pin_4), U7.10 (7)
- new net: J2.5 (Pin_5), U7.11 (6)
- new net: J2.7 (Pin_7), U7.13 (4)
- new net: J2.6 (Pin_6), U7.14 (5)
- new net: J2.10 (Pin_10), U7.15 (1)
- new net: J2.1 (Pin_1), U7.16 (0)
- new net: J2.2 (Pin_2), U7.2 (9)
- new net: U1.4 (QE), U7.3 (A)
- new net: U1.7 (QH), U7.4 (D)
- new net: U1.5 (QF), U7.6 (B)
- new net: U1.6 (QG), U7.7 (C)
- new net: J2.9 (Pin_9), U7.8 (2)
- new net: J2.8 (Pin_8), U7.9 (3)
- new net: J5.11 (Pin_11), R14.2
- new net: J6.1 (Pin_1), U2.16 (0)
- new net: J6.10 (Pin_10), U2.15 (1)
- new net: J6.11 (Pin_11), R15.2
- new net: J6.2 (Pin_2), U2.2 (9)
- new net: J6.3 (Pin_3), U2.1 (8)
- new net: J6.4 (Pin_4), U2.10 (7)
- new net: J6.5 (Pin_5), U2.11 (6)
- new net: J6.6 (Pin_6), U2.14 (5)
- new net: J6.7 (Pin_7), U2.13 (4)
- new net: J6.8 (Pin_8), U2.9 (3)
- new net: J6.9 (Pin_9), U2.8 (2)
- new net: J1.3 (Pin_3), U12.1 (8)
- new net: J1.4 (Pin_4), U12.10 (7)
- new net: J1.5 (Pin_5), U12.11 (6)
- new net: J1.7 (Pin_7), U12.13 (4)
- new net: J1.6 (Pin_6), U12.14 (5)
- new net: J1.10 (Pin_10), U12.15 (1)
- new net: J1.1 (Pin_1), U12.16 (0)
- new net: J1.2 (Pin_2), U12.2 (9)
- new net: U1.15 (QA), U12.3 (A)
- new net: U1.3 (QD), U12.4 (D)
- new net: U1.1 (QB), U12.6 (B)
- new net: U1.2 (QC), U12.7 (C)
- new net: J1.9 (Pin_9), U12.8 (2)
- new net: J1.8 (Pin_8), U12.9 (3)
- new net: R6.1, U6.10 (Rt)
- new net: C6.1, U6.11 (SS)
- new net: C8.1, U6.5 (INTVcc)
- new net: C12.2, R8.2, R9.1, U6.9 (FBX)
- new net: C9.1, D2.1 (K), D3.2 (A)
- new net: J4.1 (Pin_1), U9.16 (0)
- new net: J4.10 (Pin_10), U9.15 (1)
- new net: J4.11 (Pin_11), R13.2
- new net: J4.2 (Pin_2), U9.2 (9)
- new net: J4.3 (Pin_3), U9.1 (8)
- new net: J4.4 (Pin_4), U9.10 (7)
- new net: J4.5 (Pin_5), U9.11 (6)
- new net: J4.6 (Pin_6), U9.14 (5)
- new net: J4.7 (Pin_7), U9.13 (4)
- new net: J4.8 (Pin_8), U9.9 (3)
- new net: J4.9 (Pin_9), U9.8 (2)
- new net: J1.11 (Pin_11), R10.2
- new net: J2.11 (Pin_11), R11.2
- new net: D2.2 (A), R7.1
- new net: U10.4 (QE), U9.3 (A)
- new net: U10.7 (QH), U9.4 (D)
- new net: U10.5 (QF), U9.6 (B)
- new net: U10.6 (QG), U9.7 (C)
- new net +12V: C19.2, C4.1, C7.1, J7.1, L1.1, U4.3 (VI), U6.1 (EN/UVLO), U6.3 (Vin)
- new net +5V: A1.39 (VSYS), C1.2, C13.1, C14.2, C15.1, C16.1, C17.2, C18.1, C2.1, C3.1, C5.1, R1.1, R2.1, R3.1, R4.1, U1.10 (~{SRCLR}), U1.16 (VCC), U10.10 (~{SRCLR}), U10.16 (VCC), U11.5 (Vcc), U12.5 (Vcc), U2.5 (Vcc), U3.10 (~{SRCLR}), U3.16 (VCC), U4.2 (VO), U5.8 (VCC), U7.5 (Vcc), U8.5 (Vcc), U9.5 (Vcc)
- new net Clock: A1.15 (GPIO11), U1.11 (SRCLK), U10.11 (SRCLK), U3.11 (SRCLK)
- new net Data 1: A1.16 (GPIO12), U1.14 (SER)
- new net Data 2: U1.9 (QH'), U10.14 (SER)
- new net Data 3: U10.9 (QH'), U3.14 (SER)
- new net GND: A1.13 (GND), A1.18 (GND), A1.23 (GND), A1.28 (GND), A1.3 (GND), A1.38 (GND), A1.8 (GND), BT1.2 (-), C1.1, C11.2, C13.2, C14.1, C15.2, C16.2, C17.1, C18.2, C19.1, C2.2, C3.2, C4.2, C5.2, C6.2, C7.2, C8.2, J7.2, R5.2, R6.2, R9.2, U1.13 (~{OE}), U1.8 (GND), U10.13 (~{OE}), U10.8 (GND), U11.12 (GND), U12.12 (GND), U2.12 (GND), U3.13 (~{OE}), U3.8 (GND), U5.4 (GND), U6.12 (Mode), U6.17 (GND), U6.7 (Bias), U7.12 (GND), U8.12 (GND), U9.12 (GND)
- new net HV Out: C10.1, C12.1, D3.1 (K), R10.1, R11.1, R12.1, R13.1, R14.1, R15.1, R8.1
- new net Latch: A1.14 (GPIO10), U1.12 (RCLK), U10.12 (RCLK), U3.12 (RCLK)
- new net SCL: A1.7 (GPIO5), R2.2, U5.6 (SCL)
- new net SDA: A1.6 (GPIO4), R1.2, U5.5 (SDA)
- new net SQW: A1.9 (GPIO6), R3.2, U5.7 (SQW/OUT)
- no-connect marks 0 -> 28
Other:
- note added: "DC Input"
- note added: "Digital Logic"
- note added: "HV Boost Converter"
- note added: "Linear Voltage Regulator"
- note added: "MCU"
- note added: "RTC Module"

Commit message: edit
Parts:
- added D4: D_Schottky, Package_TO_SOT_THT:TO-220-2_Vertical, symbol Device:D_Schottky
- added D5: SMLJ13A-R, SMLJ13A-R:SMLJ13A-R, symbol SMLJ13A-R:SMLJ13A-R
- added R16: 1M, symbol Device:R
- ABS06-32.768KHZ-T1: footprint (none) -> Crystal:Crystal_SMD_MicroCrystal_CC8V-T1A-2Pin_2.0x1.2mm_HandSoldering
- BT1: footprint (none) -> Battery:BatteryHolder_Renata_SMTU2032-LF_1x2032
- C1, C14, C17: value 10nF -> 10n; footprint (none) -> Capacitor_SMD:C_0402_1005Metric_Pad0.74x0.62mm_HandSolder
- C13, C15, C16, C18, C19, C2, C3: footprint (none) -> Capacitor_SMD:C_0402_1005Metric_Pad0.74x0.62mm_HandSolder
- C4, C5: footprint (none) -> Capacitor_SMD:C_01005_0402Metric_Pad0.57x0.30mm_HandSolder
- C6: value 0.001u -> 10n
- D1, D2, D3: footprint (none) -> Package_TO_SOT_THT:TO-220-2_Vertical
- J1, J2, J3, J4, J5, J6: footprint (none) -> Connector_JST:JST_EH_B11B-EH-A_1x11_P2.50mm_Vertical
- J7: footprint (none) -> Connector_BarrelJack:BarrelJack_GCT_DCJ200-10-A_Horizontal
- R1, R2, R3: value R -> 10k; footprint (none) -> Resistor_SMD:R_0805_2012Metric_Pad1.20x1.40mm_HandSolder
- R10, R11, R12, R13, R14, R15: value 5k -> 15k; footprint (none) -> Resistor_SMD:R_0603_1608Metric_Pad0.98x0.95mm_HandSolder
- R4: footprint (none) -> Resistor_SMD:R_0402_1005Metric_Pad0.72x0.64mm_HandSolder
- R5: footprint (none) -> Resistor_SMD:R_0603_1608Metric_Pad0.98x0.95mm_HandSolder
- U1, U10, U11, U12, U2, U3, U7, U8, U9: footprint (none) -> Package_DIP:DIP-16_W7.62mm
- U6: footprint (none) -> SOP50P490X110-17N:SOP50P490X110-17N
Connections:
- net +12V: now also D4.1 (K); no longer J7.1
- net GND: now also D5.2, R16.2
- net HV Out: now also R16.1
- new net: D4.2 (A), D5.1, J7.1
- no-connect marks 28 -> 31
Other:
- moved on the sheet: BT1, C10, C11, C12, C19, C4, C5, C6, C7, C8, C9, D1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

Commit message: edit
Parts:
- removed D4: D_Schottky, Package_TO_SOT_THT:TO-220-2_Vertical, symbol Device:D_Schottky
- removed U4: LM317_SOT-223, Package_TO_SOT_SMD:SOT-223-3_TabPin2, symbol Regulator_Linear:LM317_SOT-223
- added C20: 0.1u, Capacitor_SMD:C_0402_1005Metric_Pad0.74x0.62mm_HandSolder, symbol Device:C
- added C21, C23: 0.1u, symbol Device:C
- added C22: 1u, symbol Device:C
- added C24, C25: 22u, symbol Device:C
- added FB1: FerriteBead, symbol Device:FerriteBead
- added L2: 8u, symbol Device:L
- added R17: 24.9k, symbol Device:R
- added U4: LMR33630BDDAR, LMR33630BDDAR:VREG_LM5017MR_NOPB, symbol LMR33630BDDAR:LMR33630BDDAR
- C4: value 0.1u -> 10u; footprint Capacitor_SMD:C_01005_0402Metric_Pad0.57x0.30mm_HandSolder -> (none)
- C5: value 1u -> 220n; footprint Capacitor_SMD:C_01005_0402Metric_Pad0.57x0.30mm_HandSolder -> (none)
- R10, R11, R12, R13, R14, R15: value 15k -> 10k; footprint Resistor_SMD:R_0603_1608Metric_Pad0.98x0.95mm_HandSolder -> (none)
- R4: value 240 -> 100k; footprint Resistor_SMD:R_0402_1005Metric_Pad0.72x0.64mm_HandSolder -> (none)
- R5: value 720 -> 100k; footprint Resistor_SMD:R_0603_1608Metric_Pad0.98x0.95mm_HandSolder -> (none)
Connections:
- net +12V: now also C5.1, C20.2, FB1.2, U4.2 (VIN), U4.3 (EN); no longer C19.2
- net +5V: now also R5.1, C21.1, C24.1, C25.1, L2.2; no longer C5.1, R4.1
- net GND: now also J7.MP (MountPin), C20.1, C21.2, C22.2, C24.2, C25.2, R17.2, U4.1 (PGND), U4.9 (AGND); no longer R5.2
- net at R4.2: now also U4.4 (PG); no longer R5.1
- net at D5.1, J7.1: now also C19.2, FB1.1
- new net: C22.1, R4.1, U4.6 (VCC)
- new net: R17.1, R5.2, U4.5 (FB)
- new net: C23.1, L2.1, U4.8 (SW)
- new net: C23.2, U4.7 (BOOT)
- no-connect marks 31 -> 30
Other:
- note added: "Buck Converter"
- note removed: "Linear Voltage Regulator"
- moved on the sheet: A1, ABS06-32.768KHZ-T1, BT1, C19, R1, R2, R3, U5

Commit message: edit
Parts:
- removed C19, C20: 0.1u, Capacitor_SMD:C_0402_1005Metric_Pad0.74x0.62mm_HandSolder, symbol Device:C
- removed FB1: FerriteBead, symbol Device:FerriteBead
- C10, C11: footprint (none) -> Capacitor_THT:C_Rect_L33.0mm_W20.0mm_P27.50mm_MKS4
- C12, C21, C6: footprint (none) -> Capacitor_SMD:C_0402_1005Metric_Pad0.74x0.62mm_HandSolder
- C22, C23, C5, C8: footprint (none) -> Capacitor_SMD:C_0603_1608Metric_Pad1.08x0.95mm_HandSolder
- C24, C25, C4: footprint (none) -> Capacitor_SMD:C_1210_3225Metric_Pad1.33x2.70mm_HandSolder
- C7: footprint (none) -> Capacitor_SMD:C_1206_3216Metric_Pad1.33x1.80mm_HandSolder
- C9: footprint (none) -> Capacitor_SMD:C_1206_3216Metric
- L1, L2: footprint (none) -> Inductor_SMD:L_Bourns_SRR1260
- R10: footprint (none) -> Resistor_SMD:R_0805_2012Metric_Pad1.20x1.40mm_HandSolder
- R11, R12, R13, R14, R15: footprint (none) -> Resistor_SMD:R_0815_2038Metric_Pad1.20x4.05mm_HandSolder
- R16, R8: footprint (none) -> Resistor_SMD:R_1206_3216Metric_Pad1.30x1.75mm_HandSolder
- R17, R4, R5, R6, R7, R9: footprint (none) -> Resistor_SMD:R_0603_1608Metric_Pad0.98x0.95mm_HandSolder
Connections:
- net +12V: now also D5.1, J7.1
Other:
- moved on the sheet: D5, J7
